Commit message: change dae file path

File: legged_rl_description/urdf/lite3.urdf (robot description, URDF)
Before this commit: robot lite3, 18 links, 17 joints
Links:
- link LF_calf: geometry collision box size=0.02 0.02 0.18; visual mesh filename=package://legged_rl_description/meshes/lite3/SHANK.dae
- link LF_hip: geometry visual mesh filename=package://legged_rl_description/meshes/lite3/FL_HIP.dae
- link LF_thigh: geometry collision box size=0.03 0.03 0.16; visual mesh filename=package://legged_rl_description/meshes/lite3/L_THIGH.dae
- link LH_calf: geometry collision box size=0.02 0.02 0.18; visual mesh filename=package://legged_rl_description/meshes/lite3/SHANK.dae
- link LH_hip: geometry visual mesh filename=package://legged_rl_description/meshes/lite3/HL_HIP.dae
- link LH_thigh: geometry collision box size=0.03 0.03 0.16; visual mesh filename=package://legged_rl_description/meshes/lite3/L_THIGH.dae
- link RF_calf: geometry collision box size=0.02 0.02 0.18; visual mesh filename=package://legged_rl_description/meshes/lite3/SHANK.dae
- link RF_hip: geometry visual mesh filename=package://legged_rl_description/meshes/lite3/FR_HIP.dae
- link RF_thigh: geometry collision box size=0.03 0.03 0.16; visual mesh filename=package://legged_rl_description/meshes/lite3/R_THIGH.dae
- link RH_calf: geometry collision box size=0.02 0.02 0.18; visual mesh filename=package://legged_rl_description/meshes/lite3/SHANK.dae
- link RH_hip: geometry visual mesh filename=package://legged_rl_description/meshes/lite3/HR_HIP.dae
- link RH_thigh: geometry collision box size=0.03 0.03 0.16; visual mesh filename=package://legged_rl_description/meshes/lite3/R_THIGH.dae
- link base: geometry collision box size=0.35 0.184 0.08; visual mesh filename=package://legged_rl_description/meshes/lite3/trunk.dae
