Commit message: add biped vision controller

File: legged_rl_description/urdf/biped.urdf (robot description, URDF)
Before this commit: robot biped, 10 links, 9 joints
Links:
- added link d435F_bottom_screw_frame
- added link d435F_color_frame
- added link d435F_color_optical_frame
- added link d435F_depth_frame
- added link d435F_depth_optical_frame
- added link d435F_left_ir_frame
- added link d435F_left_ir_optical_frame
- added link d435F_link, mass 0.072; collision box size=0.02505 0.09 0.025; visual mesh filename=package://realsense2_description/meshes/d435.dae
- added link d435F_right_ir_frame
- added link d435F_right_ir_optical_frame
Joints:
- added joint d435F_color_joint: type fixed, parent d435F_depth_frame, child d435F_color_frame, origin xyz=0 0.015 0 rpy=0 0 0
- added joint d435F_color_optical_joint: type fixed, parent d435F_color_frame, child d435F_color_optical_frame, origin xyz=0 0 0 rpy=-1.5707963267948966 0 -1.5707963267948966
- added joint d435F_depth_joint: type fixed, parent d435F_link, child d435F_depth_frame, origin xyz=0 0 0 rpy=0 0 0
- added joint d435F_depth_optical_joint: type fixed, parent d435F_depth_frame, child d435F_depth_optical_frame, origin xyz=0 0 0 rpy=-1.5707963267948966 0 -1.5707963267948966
- added joint d435F_joint: type fixed, parent base, child d435F_bottom_screw_frame, origin xyz=0.10 0 -0.10 rpy=0 0.69813 0
- added joint d435F_left_ir_joint: type fixed, parent d435F_depth_frame, child d435F_left_ir_frame, origin xyz=0 0.0 0 rpy=0 0 0
- added joint d435F_left_ir_optical_joint: type fixed, parent d435F_left_ir_frame, child d435F_left_ir_optical_frame, origin xyz=0 0 0 rpy=-1.5707963267948966 0 -1.5707963267948966
- added joint d435F_link_joint: type fixed, parent d435F_bottom_screw_frame, child d435F_link, origin xyz=0 0.0175 0.0125 rpy=0 0 0
- added joint d435F_right_ir_joint: type fixed, parent d435F_depth_frame, child d435F_right_ir_frame, origin xyz=0 -0.05 0 rpy=0 0 0
- added joint d435F_right_ir_optical_joint: type fixed, parent d435F_right_ir_frame, child d435F_right_ir_optical_frame, origin xyz=0 0 0 rpy=-1.5707963267948966 0 -1.5707963267948966
